File: quaver-keypad.kicad_pcb (KiCad board)
At the start: 2 copper layers, 24 parts, among them SW1 SW_Push, U1 ATmega32U4-AU, Y1 16MHz

Commit message: components placed
Parts:
- C3, C4, C5, C6, C7, F1, R1, R2, R3, R4, SW1, USB1: moved to B.Cu
- moved C4 71.6 mm to (63.1, 79.6), turned to 90 degrees
- moved SW1 69.6 mm to (48.1, 103.0), turned to 180 degrees
- moved R2 65.2 mm to (53.5, 72.2), turned to 90 degrees
- moved C7 64.5 mm to (65.9, 97.4)
- moved USB1 54.9 mm to (51.7, 61.3), turned to 270 degrees
- moved C3 53.4 mm to (58.5, 87.5), turned to 180 degrees
- moved C6 51.1 mm to (75.8, 97.4), turned to 180 degrees
- moved C5 50.2 mm to (80.5, 82.9), turned to 90 degrees
- moved R1 49.5 mm to (59.6, 79.6), turned to 90 degrees
- moved R4 46.9 mm to (80.6, 93.1), turned to 90 degrees
- moved F1 45.7 mm to (44.5, 78.4), turned to 270 degrees
- moved R3 33.3 mm to (50.0, 72.1), turned to 90 degrees
- moved C1 22.0 mm to (76.3, 72.2), turned to 90 degrees
- moved U1 12.4 mm to (70.7, 88.0)
- moved Y1 12.3 mm to (70.8, 72.2)
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
Commit message: finished general pcb
Parts:
- moved C7 8.32 mm to (58.8, 93.2), turned to 270 degrees
- moved C1 3.81 mm to (76.5, 76.0)
- moved C2 3.81 mm to (65.3, 76.0)
- moved Y1 3.80 mm to (70.9, 76.0), turned to 180 degrees
- moved R2 0.96 mm to (52.6, 71.7)
- moved R3 0.45 mm to (49.9, 71.7)
- moved R1 0.31 mm to (59.3, 79.6), turned to 270 degrees
- moved C4 0.31 mm to (62.8, 79.6)
- turned F1 to 90 degrees
- turned R4 to 270 degrees
Connections:
- U1 pad 15: Net-(U1-Pad15) -> GND
- U1 pad 23: Net-(U1-Pad15) -> GND
- U1 pad 24: Net-(U1-Pad24) -> +5V
- U1 pad 35: Net-(U1-Pad15) -> GND
- U1 pad 43: Net-(U1-Pad15) -> GND
- U1 pad 44: Net-(U1-Pad24) -> +5V
Routing:
- net GND: track 0.00 -> 163.3 mm
- net +5V: track 0.00 -> 107.4 mm, vias 0 -> 4
- net COL1: track 0.00 -> 53.2 mm
- net ROW1: track 0.00 -> 52.3 mm
- net ROW0: track 0.00 -> 50.7 mm
- net Net-(R1-Pad2): track 0.00 -> 37.0 mm, vias 0 -> 4
- net COL0: track 0.00 -> 32.7 mm
- net Net-(R3-Pad1): track 0.00 -> 29.2 mm
- net Net-(R2-Pad1): track 0.00 -> 28.3 mm
- net VCC: track 0.00 -> 13.5 mm
- net Net-(C2-Pad1): track 0.00 -> 12.9 mm
- net Net-(C1-Pad1): track 0.00 -> 10.5 mm
- net Net-(D1-Pad2): track 0.00 -> 8.32 mm
- net Net-(D2-Pad2): track 0.00 -> 8.26 mm
- net Net-(D3-Pad2): track 0.00 -> 8.14 mm
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- added copper zone on B.Cu, net GND
Other:
- net class Power added: clearance 0.2, trace_width 0.381, via_dia 0.8, via_drill 0.4
