File: quaver-keypadrev1/quaver-keypadrev1.sch (KiCad schematic (older format))
At the start: 24 parts, among them SW1 SW_Push, U1 ATmega32U4-AU, Y1 Crystal_GND24_Small

Commit message: testing controller design
Parts:
- MX1, MX2, MX3, MX4: symbol MX_Alps_Hybrid:MX-NoLED -> quaver-keypadrev1-rescue:MX-NoLED-MX_Alps_Hybrid
- USB1: symbol random-keyboard-parts:Molex-0548190589 -> quaver-keypadrev1-rescue:Molex-0548190589-random-keyboard-parts
Changed lines of the file:
@@
 EESchema Schematic File Version 4
+LIBS:quaver-keypadrev1-cache
 EELAYER 30 0
 EELAYER END
@@
 D-
 $Comp
-L random-keyboard-parts:Molex-0548190589 USB1
+L quaver-keypadrev1-rescue:Molex-0548190589-random-keyboard-parts USB1
 U 1 1 5C3480A6
 P 4075 1575
@@
 Connection ~ 5475 2475
 $Comp
-L MX_Alps_Hybrid:MX-NoLED MX4
+L quaver-keypadrev1-rescue:MX-NoLED-MX_Alps_Hybrid MX4
 U 1 1 5D09B9B4
 P 5975 3250
@@
 $EndComp
 $Comp
-L MX_Alps_Hybrid:MX-NoLED MX3
+L quaver-keypadrev1-rescue:MX-NoLED-MX_Alps_Hybrid MX3
 U 1 1 5D09AA2F
 P 5325 3250
@@
 	6125 2475 6125 3200
 $Comp
-L MX_Alps_Hybrid:MX-NoLED MX2
+L quaver-keypadrev1-rescue:MX-NoLED-MX_Alps_Hybrid MX2
 U 1 1 5D09A176
 P 5975 2525
@@
 	5475 2475 5475 3200
 $Comp
-L MX_Alps_Hybrid:MX-NoLED MX1
+L quaver-keypadrev1-rescue:MX-NoLED-MX_Alps_Hybrid MX1
 U 1 1 5D099790
 P 5325 2525
